Commit message: yaskawa: the HC10DTP's flange frame as a real one reports it
A real HC10DTP at S -24.93, L 4.27, U -23.32, R 0, B -62.41, T -155.07
read its flange, in a tool of all zeros, at 517.391, -61.828, 296.519
with Rx -180, Ry 0, Rz -180: X along base -X, Y along +Y, Z down. The
model put the flange in the same place, to 0.001 mm, but with X and Y
the other way: the guessed frame (+90 degrees about Y) turned 180
degrees about the flange's own Z. Checked at one pose; the other arms
keep the guess.

Co-Authored-By: Claude Opus 5.5 <noreply@anthropic.com>

File: src/machinist/devices/robots/urdf/yr_hc10dtp.urdf (robot description, URDF)
Before this commit: robot yr_hc10dtp, 8 links, 7 joints
Joints:
- joint joint_6_t-flange: origin xyz=0.170 0 0 rpy=0 1.5707963 0 -> xyz=0.170 0 0 rpy=0 -1.5707963 3.1415927
