Commit message: yaskawa: the GP4's flange frame as a real one reports it
A real GP4's YRC1000micro, with every joint off zero, reads its flange
(a tool of all zeros) where the GP4's model puts it, to 0.001 mm, but
turned 180 degrees about the flange's own Z from the model's guess: as
the HC10DTP's and the GP8's are.

Co-Authored-By: Claude Opus 5.5 <noreply@anthropic.com>

File: src/machinist/devices/robots/urdf/yr_gp4.urdf (robot description, URDF)
Before this commit: robot yr_gp4, 8 links, 7 joints
Joints:
- joint joint_6_t-flange: origin xyz=0.072 0 0 rpy=0 1.5707963 0 -> xyz=0.072 0 0 rpy=0 -1.5707963 3.1415927
